File: smps-filter.kicad_sch (KiCad schematic)
At the start: 13 parts, among them J1 Power IN, J2 Power OUT 1, J3 Power OUT 2, J4 Power OUT 3

Commit message: Finalied schema and PCB
Parts:
- added H1, H2, H3, H4: MountingHole_Pad, MountingHole:MountingHole_2.2mm_M2_DIN965_Pad_TopBottom, symbol Mechanical:MountingHole_Pad
- D1: footprint Diode_SMD:D_SMP_DO-220AA -> smps-filter:DO214AA
- J1, J2: footprint TerminalBlock_MetzConnect:TerminalBlock_MetzConnect_Type171_RT13702HBWC_1x02_P7.50mm_Horizontal -> smps-filter:TerminalBlock_1x02_P7.50mm_Horizontal
- L1, L2: footprint Inductor_SMD:L_10.4x10.4_H4.8 -> smps-filter:L_10.4x10.4_H4.8
Connections:
- net GND: now also H2.1, H4.1
- net Vin: now also H1.1
- net Vout: now also H3.1
Other:
- company: (none) -> ${TITLE_BLOCK_AUTHOR}
- title: (none) -> ${TITLE_BLOCK_PROJECT_NAME}
- moved on the sheet: J2, J3, J4

Commit message: Fixed DRC errors
Other:
- moved on the sheet: C1, C2, D1, H1, H2, H3, H4, J1, J2, J3, J4, L1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
